Commit message: rviz控制机械臂成功(初版)：修改urdf对应方向(未配置moveit)

File: src/m5/urdf/m5_updated_from_csv.urdf (robot description, URDF)
Before this commit: robot m5, 10 links, 9 joints
Joints:
- joint Joint2: axis -1 0 0 -> 1 0 0
- joint Joint3: axis -1 0 0 -> 1 0 0

File: src/m5_configure/config/m5.ros2_control.xacro (robot description, xacro)
@@ -2,9 +2,18 @@
 <robot xmlns:xacro="http://www.ros.org/wiki/xacro">
     <xacro:macro name="m5_ros2_control" params="name initial_positions_file">
-        <xacro:property name="initial_positions" value="${load_yaml(initial_positions_file)['initial_positions']}"/>
+        <xacro:property name="initial_positions" value="${xacro.load_yaml(initial_positions_file)['initial_positions']}"/>
         <ros2_control name="${name}" type="system">
             <hardware>
-                <!-- By default, set up controllers for simulation. This won't work on real hardware -->
-                <plugin>mock_components/GenericSystem</plugin>
+                <!-- 使用真实硬件接口连接到S3机械臂，通过UDP协议通信 -->
+                <!-- 发送角度（度），接收角度（度）并转换为弧度 -->
+                <plugin>m5_hardware/M5HardwareInterface</plugin>
+                <!-- 机械臂目标IP和端口（接收方） -->
+                <param name="robot_ip">192.168.32.150</param>
+                <param name="robot_port">7003</param>
+                <!-- 本地绑定IP和端口（发送方：电脑） -->
+                <param name="local_ip">192.168.32.135</param>
+                <param name="local_port">7001</param>
+                <param name="max_velocity">2.0</param>
+                <param name="position_tolerance">0.01</param>
             </hardware>
             <joint name="Joint1">

Commit message: 规划失败

File: src/m5/urdf/m5_updated_from_csv.urdf (robot description, URDF)
Before this commit: robot m5, 10 links, 9 joints
Links:
- removed link dummy
- added link world_link
Joints:
- removed joint dummy_joint
- added joint world_joint: type fixed, parent world_link, child base_link, origin xyz=0 0 0 rpy=0 0 0

Commit message: 重构，位置规划成功，夹爪成功控制。(MTC规划问题修复)，机械臂抖动。 1、关节限制问题修复。 2、MTC规划问题修复。 3、位置规划成功，夹爪成功控制。

File: src/m5/urdf/m5_updated_from_csv.urdf (robot description, URDF)
Before this commit: robot m5, 10 links, 9 joints
Joints:
- joint Joint1: limit lower=-3.14 upper=3.14 effort=100 velocity=1 -> lower=-6.20 upper=6.20 effort=100 velocity=1
- joint Joint2: limit lower=-1.57 upper=0 effort=100 velocity=1 -> lower=-2.97 upper=0 effort=100 velocity=1
- joint Joint3: limit lower=-1.57 upper=0 effort=100 velocity=1 -> lower=-2.97 upper=0 effort=100 velocity=1
- joint Joint4: limit lower=-3.14 upper=3.14 effort=100 velocity=1 -> lower=-6.20 upper=6.20 effort=100 velocity=1
